File: OptoInputBoard.sch (KiCad schematic (older format))
At the start: 149 parts, among them K1 CONN_3, K10 CONN_3, K11 CONN_3, K12 CONN_3, K13 CONN_3, K14 CONN_3, K15 CONN_3, K16 CONN_3, K17 CONN_3, K18 CONN_3, K19 CONN_3, K2 CONN_3, K3 CONN_3, K4 CONN_3, K5 CONN_3, K6 CONN_3, K7 CONN_3, K8 CONN_3, K9 CONN_3, P1 CONN_20, U1 4N25, U10 74HC04, U11 74HC04, U12 4N25, U13 4N25, U14 4N25, U15 4N25, U16 4N25, U17 4N25, U18 4N25, U19 4N25, U2 4N25, U20 4N25, U21 74HC04, U3 4N25, U4 4N25, U5 4N25, U6 4N25, U7 4N25, U8 4N25, U9 4N25

Commit message: saved with new kicad version
Parts:
- C1, C10, C11, C12, C13, C14, C15, C16, C17, C18, C2, C3, C4, C5, C6, C7, C8, C9: footprint (none) -> Capacitors_ThroughHole:Capacitor6MMDiscRM5
- D1, D19, D2, D20, D21, D22, D23, D24, D25, D26, D27, D3, D4, D5, D6, D7, D8, D9: footprint (none) -> Diodes_ThroughHole:Diode_DO-41_SOD81_Horizontal_RM10
- D10, D11, D12, D13, D14, D15, D16, D17, D18, D28, D29, D30, D31, D32, D33, D34, D35, D36: footprint (none) -> LEDs:LED-3MM
- K1, K10, K11, K12, K13, K14, K15, K16, K17, K18, K19, K2, K3, K4, K5, K6, K7, K8, K9: footprint (none) -> Pin_Headers:Pin_Header_Straight_1x03
- P1: footprint (none) -> Pin_Headers:Pin_Header_Straight_1x20
- R1, R10, R11, R12, R13, R14, R15, R16, R17, R18, R19, R2, R20, R21, R22, R23, R24, R25, R26, R27, R28, R29, R3, R30, R31, R32, R33, R34, R35, R36, R37, R38, R39, R4, R40, R41, R42, R43, R44, R45, R46, R47, R48, R49, R5, R50, R51, R52, R53, R54, R6, R7, R8, R9: footprint (none) -> Resistors_ThroughHole:Resistor_Horizontal_RM10mm
- U1, U12, U13, U14, U15, U16, U17, U18, U19, U2, U20, U3, U4, U5, U6, U7, U8, U9: footprint (none) -> Sockets_DIP:DIP-6__300
- U10, U11, U21: footprint (none) -> Sockets_DIP:DIP-14__300
